File: Código Fuente/Exquisite Lahdi-Borwo.brd (EAGLE design)
At the start: 56.8 x 53.3 mm, 28 parts, among them P1 10V, P2 10V, P3 10V

Commit message: Inicio
Parts:
- removed Meter10, Meter11, Meter12, Meter14, Meter15, Meter16, Meter2, Meter6: (no value), AUTODESK_CIRCUITS_BREADBOARD:DC-POWER
- removed P1, P2, P3: 10V, AUTODESK_CIRCUITS_BREADBOARD:2P-2.54-65/35MIL
- removed R10, R13: 3.9k‎Ω, AUTODESK_CIRCUITS_BREADBOARD:0207/10
- removed R11, R9: 1k‎Ω, AUTODESK_CIRCUITS_BREADBOARD:0207/10
- removed R12, R14, R3, R4, R8: 2.2k‎Ω, AUTODESK_CIRCUITS_BREADBOARD:0207/10
- removed R15, R6, R7: 1.8k‎Ω, AUTODESK_CIRCUITS_BREADBOARD:0207/10
- added C1, C2: 10uF, AUTODESK_CIRCUITS_BREADBOARD:C5B2.5
- added FUNC1, FUNC2: (no value), AUTODESK_CIRCUITS_BREADBOARD:DC-POWER
- added L2: 100mH, AUTODESK_CIRCUITS_BREADBOARD:0207/10
- L1: value 2.2k‎Ω -> 100mH
- R1: value 1k‎Ω -> 100‎Ω
- R2: value 3.9k‎Ω -> 100‎Ω
- moved R1 50.8 mm to (5.00, 10.1)
- moved Meter4 25.4 mm to (5.00, 124.4)
- moved R2 12.7 mm to (5.00, 86.3)
- renumbered Meter5 to Meter3, R5 to L1
Connections:
- removed net N$10: Meter11.-, R8.2
- removed net N$11: Meter12.-, P1.1
- removed net N$12: Meter10.+, R10.1, R8.1
- removed net N$13: Meter15.-, R9.1
- removed net N$14: Meter14.-, R10.2
- removed net N$15: Meter15.+, P1.2
- removed net N$16: R11.2, R12.1, R13.2
- removed net N$17: R12.2, R14.2
- removed net N$18: R13.1, R14.1, R15.2
- removed net N$19: P3.1, R15.1
- removed net N$20: P3.2, R11.1
- removed net N$7: Meter12.+, R6.1
- removed net N$8: Meter11.+, R4.2
- removed net N$9: Meter10.-, R6.2
- net N$1: now also FUNC2.-, L1.1, L2.2; no longer Meter16.+, Meter2.-, R1.2, R2.2, R3.1
- net N$2: now also L1.2, L2.1, Meter4.-, R2.2; no longer Meter2.+, P2.2, R1.1
- net N$3: now also FUNC2.+; no longer L1.1, Meter3.-, Meter4.-, Meter6.+, R7.2
- net N$4: now also FUNC1.+, R1.1; no longer Meter6.-, P2.1, R7.1
- net N$5: now also C1.1, C2.2, FUNC1.-; no longer L1.2, Meter16.-, R3.2
- net N$6: now also C1.2, C2.1, Meter3.-, R1.2; no longer Meter14.+, R4.1, R9.2
